File: c64_orchestra/destination_control.sch (KiCad schematic (older format))
At the start: 4 parts

Commit message: Added parts of schematic and worked on pcb layout.
Parts:
- U5: renamed from U?; footprint (none) -> Package_DIP:DIP-14_W7.62mm
- U6, U7: renamed from U?; footprint (none) -> Package_DIP:DIP-20_W7.62mm
Changed lines of the file:
@@
 Global_GND
 $Comp
-L 74xx:74HC374 U?
+L 74xx:74HC374 U6
 U 1 1 5F9DAC92
 P 5650 1900
-F 0 "U?" H 5650 2881 50  0000 C CNN
+F 0 "U6" H 5650 2881 50  0000 C CNN
 F 1 "74HC374" H 5650 2790 50  0000 C CNN
-F 2 "" H 5650 1900 50  0001 C CNN
+F 2 "Package_DIP:DIP-20_W7.62mm" H 5650 1900 50  0001 C CNN
 F 3 "https://www.ti.com/lit/ds/symlink/cd74hct374.pdf" H 5650 1900 50  0001 C CNN
 	1    5650 1900
@@
 	4400 1800 5150 1800
 $Comp
-L 74xx:74HC374 U?
+L 74xx:74HC374 U7
 U 1 1 5F9DEED7
 P 5650 3750
-F 0 "U?" H 5650 4731 50  0000 C CNN
+F 0 "U7" H 5650 4731 50  0000 C CNN
 F 1 "74HC374" H 5650 4640 50  0000 C CNN
-F 2 "" H 5650 3750 50  0001 C CNN
+F 2 "Package_DIP:DIP-20_W7.62mm" H 5650 3750 50  0001 C CNN
 F 3 "https://www.ti.com/lit/ds/symlink/cd74hct374.pdf" H 5650 3750 50  0001 C CNN
 	1    5650 3750
@@
 	1800 3800 4950 3800
 $Comp
-L 74xx_IEEE:7408 U?
+L 74xx_IEEE:7408 U5
 U 1 1 5FA382F7
 P 2900 2800
-F 0 "U?" H 2900 3216 50  0000 C CNN
+F 0 "U5" H 2900 3216 50  0000 C CNN
 F 1 "7408" H 2900 3125 50  0000 C CNN
-F 2 "" H 2900 2800 50  0001 C CNN
+F 2 "Package_DIP:DIP-14_W7.62mm" H 2900 2800 50  0001 C CNN
 F 3 "" H 2900 2800 50  0001 C CNN
 	1    2900 2800
@@
 	2050 2700 2350 2700
 $Comp
-L 74xx_IEEE:7408 U?
+L 74xx_IEEE:7408 U5
 U 2 1 5FA3A92D
 P 2900 3350
-F 0 "U?" H 2900 3766 50  0000 C CNN
+F 0 "U5" H 2900 3766 50  0000 C CNN
 F 1 "7408" H 2900 3675 50  0000 C CNN
-F 2 "" H 2900 3350 50  0001 C CNN
+F 2 "Package_DIP:DIP-14_W7.62mm" H 2900 3350 50  0001 C CNN
 F 3 "" H 2900 3350 50  0001 C CNN
 	2    2900 3350
